Commit message: 2nd commit

File: urdf/amr_base.xacro (robot description, xacro)
@@ -3,13 +3,14 @@
     <!--************* CONSTANTS **************-->
     <!-- Define the robot's dimensions -->
-    <xacro:property name="robot_radius" value="0.23" />
+    <!--<xacro:property name="robot_radius" value="0.23" />-->
     <xacro:property name="wheel_radius" value="0.0825" />
     <xacro:property name="wheel_width" value="0.0435" />
     <xacro:property name="wheel_base" value="0.365" />
     <xacro:property name="base_height" value="0.255" />
+    <!--<xacro:property name="pi" value="3.1415927" />-->
     <!-- Define intertia macros  -->
     <xacro:macro name="box_inertia" params="m w h d">
         <inertial>
-            <origin xyz="0 0 0" rpy="${pi/2} 0 ${pi/2}" />
+            <origin xyz="0 0 0" rpy="1.57 0 1.57" />
             <mass value="${m}" />
             <inertia ixx="${(m/12) * (h*h + d*d)}" ixy="0.0" ixz="0.0" iyy="${(m/12) * (w*w + d*d)}" iyz="0.0" izz="${(m/12) * (w*w + h*h)}" />
@@ -18,5 +19,5 @@
     <xacro:macro name="cylinder_inertia" params="m r h">
         <inertial>
-            <origin xyz="0 0 0" rpy="${pi/2} 0 0" />
+            <origin xyz="0 0 0" rpy="1.57 0 0" />
             <mass value="${m}" />
             <inertia ixx="${(m/12) * (3*r*r + h*h)}" ixy="0" ixz="0" iyy="${(m/12) * (3*r*r + h*h)}" iyz="0" izz="${(m/2) * (r*r)}" />
@@ -40,7 +41,7 @@
         <visual>
             <geometry>
-                <mesh filename="file:///home/mauro/amr_ws/src/amr_desc/meshes/amr_base.dae" />
-            </geometry>
-            <origin rpy="0 0 ${pi/2}" xyz="0 0 0.033" />
+                <mesh filename="file:///home/jpalves/ros2_ws/src/robot1/models/amr/meshes/ROBOTSEMNADA.dae" />
+            </geometry>
+            <origin rpy="0 0 1.5708" xyz="0.235 0.025 0.033" />
             <material name="metal">
                 <color rgba="0.8 0.8 0.8 1" />
@@ -50,8 +51,30 @@
             <origin rpy="0 0 0" xyz="0 0 0.1625" />
             <geometry>
-                <cylinder radius="${robot_radius}" length="0.255" />
+                <cylinder radius="0.23" length="0.255" />
             </geometry>
         </collision>
-        <xacro:cylinder_inertia m="40000.0" r="${robot_radius}" h="0.255" />
+        <xacro:cylinder_inertia m="40.0302" r="0.23" h="0.255" />
+    </link>
+    <joint name="base_to_torre" type="fixed">
+    	<origin xyz="0 0 0.285" rpy="0 0 1.5708" />
+    	<parent link="base_link" />
+    	<child link="torre_link" />
+    </joint>
+    <link name="torre_link">
+    	   <visual>
+                <origin xyz="0 0 0.285" rpy="0 0 0" />
+                <geometry>
+                    <mesh filename="file:///home/jpalves/ros2_ws/src/robot1/models/amr/meshes/torre001.dae" />
+                </geometry>
+                <material name="black">
+                    <color rgba="0 0 0 1" />
+                </material>
+            </visual>
+            <collision>
+                <origin xyz="0 0 0.285" rpy="0 0 0" />
+                <geometry>
+                    <mesh filename="file:///home/jpalves/ros2_ws/src/robot1/models/amr/meshes/torre001.dae" />
+                </geometry>
+            </collision>
     </link>
     <!--************* ROBOT'S WHEELS **************-->
@@ -59,7 +82,7 @@
         <link name="${prefix}_link">
             <visual>
-                <origin xyz="0 0 0" rpy="${pi/2} 0 0" />
-                <geometry>
-                    <mesh filename="file:///home/mauro/amr_ws/src/amr_desc/meshes/amr_wheel.dae" />
+                <origin xyz="0 0 0" rpy="1.57 0 0" />
+                <geometry>
+                    <mesh filename="file:///home/jpalves/ros2_ws/src/robot1/models/amr/meshes/amr_wheel.dae" />
                 </geometry>
                 <material name="black">
@@ -78,5 +101,5 @@
             <parent link="base_link" />
             <child link="${prefix}_link" />
-            <origin xyz="0 ${reflect*(wheel_base/2)} ${wheel_radius}" rpy="${-reflect * (pi/2)} 0 0" />
+            <origin xyz="0 ${reflect*(wheel_base/2)} ${wheel_radius}" rpy="${-reflect * 1.57} 0 0" />
             <limit upper="0" lower="0" effort="1" velocity="5.0" />
             <axis xyz="0 0 ${reflect}" />
@@ -90,7 +113,8 @@
             <visual>
                 <geometry>
-                    <mesh filename="file:///home/mauro/amr_ws/src/amr_desc/meshes/amr_caster.dae" />
-                </geometry>
-                <origin rpy="0 0 ${pi/2}" xyz="0 0 0" />
+                    <sphere radius="0.025"/>
+                    <!--<mesh filename="file:///home/jpalves/ros2_ws/src/robot1/models/amr/meshes/amr_caster.dae" />-->
+                </geometry>
+                <origin rpy="0 0 1.57" xyz="0 0 0" />
                 <material name="white">
                     <color rgba="1 1 1 1" />
@@ -98,7 +122,7 @@
             </visual>
             <collision>
-                <origin xyz="0 0 ${wheel_radius/2}" rpy="0 0 0" />
-                <geometry>
-                    <sphere radius="${0.108/2}" />
+                <origin xyz="0 0 0.025" rpy="0 0 0" />
+                <geometry>
+                    <sphere radius="0.025" />
                 </geometry>
             </collision>
@@ -114,7 +138,7 @@
     <xacro:caster prefix="fcaster" position="0.135 0 0" />
     <xacro:caster prefix="lcaster" position="-0.135 0.105 0" />
-    <xacro:caster prefix="rcaster" position="-0.135 -0.105 0" />
+    <!--<xacro:caster prefix="rcaster" position="-0.135 -0.105 0" />-->
     <!--************* ROBOT'S LASER **************-->
-    <link name="laser">
+    <link name="base_scan">
         <visual>
             <geometry>
@@ -129,5 +153,5 @@
     <joint name="base_to_scanner" type="fixed">
         <parent link="base_link" />
-        <child link="laser" />
+        <child link="base_scan" />
         <origin xyz="0.165 0 0.24" rpy="0 0 0" />
     </joint>
@@ -136,7 +160,7 @@
         <visual>
             <geometry>
-                <mesh filename="file:///home/mauro/amr_ws/src/amr_desc/meshes/d435.dae" />
-            </geometry>
-            <origin rpy="${pi/2} 0 ${pi/2}" xyz="0 0 0" />
+                <mesh filename="file:///home/jpalves/ros2_ws/src/robot1/models/amr/meshes/d435.dae" />
+            </geometry>
+            <origin rpy="1.57 0 1.57" xyz="0 0 0" />
             <material name="black">
                 <color rgba="0 0 0 1" />
@@ -144,14 +168,72 @@
         </visual>
     </link>
-    <joint name="base_to_camera" type="fixed">
+    <joint name="camera_joint" type="fixed">
         <parent link="base_link" />
         <child link="camera_link" />
         <origin rpy="0 0 0" xyz="0.23 0 0.15" />
     </joint>
-    <link name="imu_link" />
-    <joint name="imu_joint" type="fixed">
+    <joint name="camera_rgb_joint" type="fixed">
+    	<origin xyz="0.00 0.0 0.0" rpy="0 0 0"/>
+    	<!-- <origin xyz="${r200_cam_rgb_px} ${r200_cam_rgb_py} ${r200_cam_rgb_pz}" rpy="0 0 0"/> -->
+    	<parent link="camera_link"/>
+    	<child link="camera_rgb_frame"/>
+    </joint>
+    <link name="camera_rgb_frame"/>
+    <joint name="camera_rgb_optical_joint" type="fixed">
+         <origin xyz="0 0 0" rpy="-1.57 0 -1.57"/>
+         <parent link="camera_rgb_frame"/>
+         <child link="camera_rgb_optical_frame"/>
+   </joint>
+  <link name="camera_rgb_optical_frame"/>
+  <link name="imu_link" />
+  <joint name="imu_joint" type="fixed">
         <parent link="camera_link" />
         <child link="imu_link" />
         <origin rpy="0 0 0" xyz="0 0 0" />
-    </joint>
+  </joint>
+  <link name="camera_depth_frame"></link>
+  <link name="camera_depth_optical_frame"></link>
+  <joint name="camera_depth_joint" type="fixed">
+    <parent link="camera_link" />
+    <child link="camera_depth_frame" />
+    <pose xyz="0 0 0" rpy="0 0 0" />
+  </joint>
+  <joint name="camera_depth_optical_joint" type="fixed">
+    <parent link="camera_depth_frame" />
+    <child link="camera_depth_optical_frame" />
+    <pose xyz="0 0 0 " rpy="-1.57 0 -1.57" />
+  </joint>
+  <!-- *********************** WHEEL ODOMETRY ***************************    -->
+  <gazebo>
+    <plugin name="amr_diff_drive" filename="amr_diff_drive.so">
+      <update_rate>30</update_rate>
+      <!-- wheels -->
+      <left_joint>lwheel_joint</left_joint>
+      <right_joint>rwheel_joint</right_joint>
+      <!-- kinematics -->
+      <wheel_separation>0.365</wheel_separation>
+      <wheel_diameter>0.165</wheel_diameter>
+      <!-- limits -->
+      <max_wheel_torque>200</max_wheel_torque>
+      <max_wheel_acceleration>1.0</max_wheel_acceleration>
+      <!-- Receive velocity commands on this ROS topic -->
+      <command_topic>cmd_vel</command_topic>
+      <!-- output -->
+      <!-- When false, publish no wheel odometry data to a ROS topic -->
+      <publish_odom>true</publish_odom>
+      <!-- When true, publish coordinate transform from odom to base_footprint -->
+      <!-- I usually use the robot_localization package to publish this transform -->
+      <publish_odom_tf>false</publish_odom_tf>
+      <!-- When true, publish coordinate transform from base_link to the wheels -->
+      <!-- The robot_state_publisher package is often used to publish this transform -->
+      <publish_wheel_tf>true</publish_wheel_tf>
+      <odometry_topic>odometry</odometry_topic>
+      <odometry_frame>odom</odometry_frame>
+      <robot_base_frame>base_link</robot_base_frame>
+      <odometry_source>1</odometry_source>
+      <!--<ros>
+        <remapping>odom:=wheel/odometry</remapping>
+      </ros>-->
+    </plugin>
+  </gazebo>
 </robot>

File: urdf/jetracer.xacro (robot description, xacro)
@@ -117,5 +117,5 @@
         <parent link="base_link" />
         <child link="base_scan" />
-        <origin xyz="0 0 0" rpy="0 0 0" />
+        <origin xyz="0.165 0 0.24" rpy="0 0 0" />
     </joint>
   <link name="rr_wheel">
